File: PCMTester2.0/PCMTester2.0.kicad_sch (KiCad schematic)
At the start: 63 parts

Commit message: adding new design footprints and schematic
Parts:
- C1, C2, C3, C4, C5, C6: footprint CAPC2012X135N -> PCMTester2.0 Footprints:22uF_Capacitor
- DF12: footprint HRS_DF12NB-60DS-0.5V(51) -> PCMTester2.0 Footprints:HRS_DF12NB-60DS-0.5V_51_
- J_COMPAT1, J_EXTEND1: footprint SAMTEC_QTH-040-01-L-D-DP-A -> PCMTester2.0 Footprints:SAMTEC_QTH-040-01-X-D-DP-A
- NT_01_N1, NT_01_P1, NT_02_N1, NT_02_P1, NT_03_N1, NT_03_P1, NT_04_N1, NT_04_P1, NT_05_N1, NT_05_P1, NT_06_N1, NT_06_P1, NT_07_N1, NT_07_P1, NT_08_N1, NT_08_P1, NT_09_N1, NT_09_P1, NT_10_N1, NT_10_P1, NT_11_N1, NT_11_P1, NT_12_N1, NT_12_P1, NT_14_N1, NT_14_P1, NT_18_N1, NT_18_P1, NT_20_N1, NT_20_P1, NT_21_N1, NT_21_P1, NT_22_N1, NT_22_P1, NT_23_N1, NT_23_P1, NT_24_N1, NT_24_P1, NT_27_N1, NT_27_P1, NT_28_N1, NT_28_P1: footprint Net_Tie1 -> (none)
- PWR_CORE1: footprint PHOENIX_1988105 - duplicate -> PCMTester2.0 Footprints:PWR_CORE1_footprint
- R1, R2, R3, R4, R5, R6: footprint RESC1608X55X30LL15T15 -> PCMTester2.0 Footprints:RESC1608X50N
- TO_BM1: footprint HIROSE_FX11A-80P-8-SV -> PCMTester2.0 Footprints:TO_BM1_footprint
- TP1, TP2, TP3, TP_VBRD1: footprint CONN HEADER 1POS .100_ -> PCMTester2.0 Footprints:SAMTEC_TSW-101-07-G-S (pin)
Changed lines of the file:
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@@
 			)
 		)
-		(property "Footprint" "Net_Tie1"
+		(property "Footprint" ""
 			(at 497.84 114.3 0)
 			(effects
@@
 			)
 		)
-		(property "Footprint" "Net_Tie1"
+		(property "Footprint" ""
 			(at 354.33 215.9 0)
 			(effects
@@
 			)
 		)
-		(property "Footprint" "Net_Tie1"
+		(property "Footprint" ""
 			(at 288.29 220.98 0)
 			(effects
@@
 			)
 		)
-		(property "Footprint" "Net_Tie1"
+		(property "Footprint" ""
 			(at 288.29 208.28 0)
 			(effects
@@
 			)
 		)
-		(property "Footprint" "CAPC2012X135N"
+		(property "Footprint" "PCMTester2.0 Footprints:22uF_Capacitor"
 			(at 44.45 83.82 0)
 			(effects
@@
 			)
 		)
-		(property "Footprint" "Net_Tie1"
+		(property "Footprint" ""
 			(at 288.29 238.76 0)
 			(effects
@@
 			)
 		)
-		(property "Footprint" "Net_Tie1"
+		(property "Footprint" ""
 			(at 288.29 236.22 0)
 			(effects
@@
 			)
 		)
-		(property "Footprint" "Net_Tie1"
+		(property "Footprint" ""
 			(at 497.84 104.14 0)
 			(effects
@@
 			)
 		)
-		(property "Footprint" "Net_Tie1"
+		(property "Footprint" ""
 			(at 288.29 200.66 0)
 			(effects
@@
 			)
 		)
-		(property "Footprint" "Net_Tie1"
+		(property "Footprint" ""
 			(at 496.57 152.4 0)
 			(effects
@@
 			)
 		)
-		(property "Footprint" "Net_Tie1"
+		(property "Footprint" ""
 			(at 497.84 127 0)
 			(effects
@@
 			)
 		)
-		(property "Footprint" "Net_Tie1"
+		(property "Footprint" ""
 			(at 288.29 228.6 0)
 			(effects
@@
 			)
 		)
-		(property "Footprint" "Net_Tie1"
+		(property "Footprint" ""
 			(at 497.84 121.92 0)
 			(effects
@@
 			)
 		)
-		(property "Footprint" "CONN HEADER 1POS .100_"
+		(property "Footprint" "PCMTester2.0 Footprints:SAMTEC_TSW-101-07-G-S (pin)"
 			(at 162.56 300.99 0)
 			(effects
@@
 			)
 		)
-		(property "Footprint" "RESC1608X55X30LL15T15"
+		(property "Footprint" "PCMTester2.0 Footprints:RESC1608X50N"
 			(at 116.84 34.29 0)
 			(effects
@@
 			)
 		)
-		(property "Footprint" "CAPC2012X135N"
+		(property "Footprint" "PCMTester2.0 Footprints:22uF_Capacitor"
 			(at 55.88 265.43 0)
 			(effects
@@
 			)
 		)
-		(property "Footprint" "Net_Tie1"
+		(property "Footprint" ""
 			(at 354.33 213.36 0)
 			(effects
@@
 			)
 		)
-		(property "Footprint" "Net_Tie1"
+		(property "Footprint" ""
 			(at 497.84 111.76 0)
 			(effects
@@
 			)
 		)
-		(property "Footprint" "Net_Tie1"
+		(property "Footprint" ""
 			(at 496.57 144.78 0)
 			(effects
@@
 			)
 		)
-		(property "Footprint" "CAPC2012X135N"
+		(property "Footprint" "PCMTester2.0 Footprints:22uF_Capacitor"
 			(at 48.26 111.76 0)
 			(effects
@@
 			)
 		)
-		(property "Footprint" "Net_Tie1"
+		(property "Footprint" ""
 			(at 497.84 119.38 0)
 			(effects
@@
 			)
 		)
-		(property "Footprint" "PHOENIX_1988105 - duplicate"
+		(property "Footprint" "PCMTester2.0 Footprints:PWR_CORE1_footprint"
 			(at 39.37 119.38 0)
 			(effects
@@
 			)
 		)
-		(property "Footprint" "CONN HEADER 1POS .100_"
+		(property "Footprint" "PCMTester2.0 Footprints:SAMTEC_TSW-101-07-G-S (pin)"
 			(at 356.87 114.3 0)
 			(effects
@@
 			)
 		)
-		(property "Footprint" "Net_Tie1"
+		(property "Footprint" ""
 			(at 288.29 213.36 0)
 			(effects
@@
 			)
 		)
-		(property "Footprint" "CONN HEADER 1POS .100_"
+		(property "Footprint" "PCMTester2.0 Footprints:SAMTEC_TSW-101-07-G-S (pin)"
 			(at 375.92 177.8 0)
 			(effects
@@
 			)
 		)
-		(property "Footprint" "Net_Tie1"
+		(property "Footprint" ""
 			(at 288.29 198.12 0)
 			(effects
@@
 			)
 		)
-		(property "Footprint" "Net_Tie1"
+		(property "Footprint" ""
 			(at 497.84 129.54 0)
 			(effects
@@
 			)
 		)
-		(property "Footprint" "CAPC2012X135N"
+		(property "Footprint" "PCMTester2.0 Footprints:22uF_Capacitor"
 			(at 35.56 83.82 0)
 			(effects
@@
 			)
 		)
-		(property "Footprint" "RESC1608X55X30LL15T15"
+		(property "Footprint" "PCMTester2.0 Footprints:RESC1608X50N"
 			(at 134.62 48.26 0)
 			(effects
@@
 			)
 		)
-		(property "Footprint" "SAMTEC_QTH-040-01-L-D-DP-A"
+		(property "Footprint" "PCMTester2.0 Footprints:SAMTEC_QTH-040-01-X-D-DP-A"
 			(at 455.93 104.14 0)
 			(effects
@@
 			)
 		)
-		(property "Footprint" "Net_Tie1"
+		(property "Footprint" ""
 			(at 496.57 142.24 0)
 			(effects
@@
 			)
 		)
-		(property "Footprint" "Net_Tie1"
+		(property "Footprint" ""
 			(at 496.57 157.48 0)
 			(effects
@@
 			)
 		)
-		(property "Footprint" "CAPC2012X135N"
+		(property "Footprint" "PCMTester2.0 Footprints:22uF_Capacitor"
 			(at 55.88 274.32 0)
 			(effects
@@
 			)
 		)
-		(property "Footprint" "Net_Tie1"
+		(property "Footprint" ""
 			(at 288.29 223.52 0)
 			(effects
@@
 			)
 		)
-		(property "Footprint" "Net_Tie1"
+		(property "Footprint" ""
 			(at 496.57 160.02 0)
 			(effects
@@
 			)
 		)
-		(property "Footprint" "Net_Tie1"
+		(property "Footprint" ""
 			(at 354.33 223.52 0)
 			(effects
@@
 			)
 		)
-		(property "Footprint" "CONN HEADER 1POS .100_"
+		(property "Footprint" "PCMTester2.0 Footprints:SAMTEC_TSW-101-07-G-S (pin)"
 			(at 267.97 177.8 0)
 			(effects
@@
 			)
 		)
-		(property "Footprint" "Net_Tie1"
+		(property "Footprint" ""
 			(at 288.29 182.88 0)
 			(effects
@@
 			)
 		)
-		(property "Footprint" "Net_Tie1"
+		(property "Footprint" ""
 			(at 288.29 190.5 0)
 			(effects
@@
 			)
 		)
-		(property "Footprint" "RESC1608X55X30LL15T15"
+		(property "Footprint" "PCMTester2.0 Footprints:RESC1608X50N"
 			(at 116.84 29.21 0)
 			(effects
@@
 			)
 		)
-		(property "Footprint" "Net_Tie1"
+		(property "Footprint" ""
 			(at 354.33 220.98 0)
 			(effects
@@
 			)
 		)
-		(property "Footprint" "Net_Tie1"
+		(property "Footprint" ""
 			(at 496.57 149.86 0)
 			(effects
@@
 			)
 		)
-		(property "Footprint" "HIROSE_FX11A-80P-8-SV"
+		(property "Footprint" "PCMTester2.0 Footprints:TO_BM1_footprint"
 			(at 110.49 232.41 0)
 			(effects
@@
 			)
 		)
-		(property "Footprint" "Net_Tie1"
+		(property "Footprint" ""
 			(at 288.29 254 0)
 			(effects
@@
 			)
 		)
-		(property "Footprint" "CAPC2012X135N"
+		(property "Footprint" "PCMTester2.0 Footprints:22uF_Capacitor"
 			(at 57.15 111.76 0)
 			(effects
@@
 			)
 		)
-		(property "Footprint" "RESC1608X55X30LL15T15"
+		(property "Footprint" "PCMTester2.0 Footprints:RESC1608X50N"
 			(at 134.62 63.5 0)
 			(effects
@@
 			)
 		)
-		(property "Footprint" "Net_Tie1"
+		(property "Footprint" ""
 			(at 354.33 205.74 0)
 			(effects
@@
 			)
 		)
-		(property "Footprint" "Net_Tie1"
+		(property "Footprint" ""
 			(at 288.29 205.74 0)
 			(effects
@@
 			)
 		)
-		(property "Footprint" "SAMTEC_QTH-040-01-L-D-DP-A"
+		(property "Footprint" "PCMTester2.0 Footprints:SAMTEC_QTH-040-01-X-D-DP-A"
 			(at 313.69 106.68 0)
 			(effects
@@
 			)
 		)
-		(property "Footprint" "RESC1608X55X30LL15T15"
+		(property "Footprint" "PCMTester2.0 Footprints:RESC1608X50N"
 			(at 134.62 53.34 0)
 			(effects
@@
 			)
 		)
-		(property "Footprint" "Net_Tie1"
+		(property "Footprint" ""
 			(at 354.33 231.14 0)
 			(effects
@@
 			)
 		)
-		(property "Footprint" "Net_Tie1"
+		(property "Footprint" ""
 			(at 288.29 185.42 0)
 			(effects
@@
 			)
 		)
-		(property "Footprint" "Net_Tie1"
+		(property "Footprint" ""
 			(at 288.29 246.38 0)
 			(effects
@@
 			)
 		)
-		(property "Footprint" "Net_Tie1"
+		(property "Footprint" ""
 			(at 354.33 208.28 0)
 			(effects
@@
 			)
 		)
-		(property "Footprint" "Net_Tie1"
+		(property "Footprint" ""
 			(at 288.29 231.14 0)
 			(effects
@@
 			)
 		)
-		(property "Footprint" "Net_Tie1"
+		(property "Footprint" ""
 			(at 288.29 251.46 0)
 			(effects
@@
 			)
 		)
-		(property "Footprint" "Net_Tie1"
+		(property "Footprint" ""
 			(at 288.29 193.04 0)
 			(effects
@@
 			)
 		)
-		(property "Footprint" "HRS_DF12NB-60DS-0.5V(51)"
+		(property "Footprint" "PCMTester2.0 Footprints:HRS_DF12NB-60DS-0.5V_51_"
 			(at 85.09 99.06 0)
 			(effects
@@
 			)
 		)
-		(property "Footprint" "Net_Tie1"
+		(property "Footprint" ""
 			(at 288.29 243.84 0)
 			(effects
@@
 			)
 		)
-		(property "Footprint" "RESC1608X55X30LL15T15"
+		(property "Footprint" "PCMTester2.0 Footprints:RESC1608X50N"
 			(at 134.62 58.42 0)
 			(effects
@@
 			)
 		)
-		(property "Footprint" "Net_Tie1"
+		(property "Footprint" ""
 			(at 497.84 106.68 0)
 			(effects
@@
 			)
 		)
-		(property "Footprint" "Net_Tie1"
+		(property "Footprint" ""
 			(at 288.29 215.9 0)
 			(effects
@@
 			)
 		)
-		(property "Footprint" "Net_Tie1"
+		(property "Footprint" ""
 			(at 354.33 228.6 0)
 			(effects

Commit message: new pcb design with components laid out
Parts:
- C1, C2, C3, C4, C5, C6: footprint PCMTester2.0 Footprints:22uF_Capacitor -> PCMFootprints:22uF_Capacitor
- DF12: footprint PCMTester2.0 Footprints:HRS_DF12NB-60DS-0.5V_51_ -> PCMFootprints:HRS_DF12NB-60DS-0.5V_51_
- J_COMPAT1, J_EXTEND1: footprint PCMTester2.0 Footprints:SAMTEC_QTH-040-01-X-D-DP-A -> PCMFootprints:SAMTEC_QTH-040-01-X-D-DP-A
- PWR_CORE1: footprint PCMTester2.0 Footprints:PWR_CORE1_footprint -> PCMTester2.0_Footprints:PWR_CORE1_footprint
- R1, R2, R3, R4, R5, R6: footprint PCMTester2.0 Footprints:RESC1608X50N -> PCMTester2.0_Footprints:RESC1608X50N
- TO_BM1: footprint PCMTester2.0 Footprints:TO_BM1_footprint -> PCMTester2.0_Footprints:TO_BM1_footprint
- TP1, TP2, TP3, TP_VBRD1: footprint PCMTester2.0 Footprints:SAMTEC_TSW-101-07-G-S (pin) -> PCMFootprints:SAMTEC_TSW-101-07-G-S (pin)
Changed lines of the file:
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@@
 			)
 		)
-		(property "Footprint" "PCMTester2.0 Footprints:22uF_Capacitor"
+		(property "Footprint" "PCMFootprints:22uF_Capacitor"
 			(at 44.45 83.82 0)
 			(effects
@@
 			)
 		)
-		(property "Footprint" "PCMTester2.0 Footprints:SAMTEC_TSW-101-07-G-S (pin)"
+		(property "Footprint" "PCMFootprints:SAMTEC_TSW-101-07-G-S (pin)"
 			(at 162.56 300.99 0)
 			(effects
@@
 			)
 		)
-		(property "Footprint" "PCMTester2.0 Footprints:RESC1608X50N"
+		(property "Footprint" "PCMTester2.0_Footprints:RESC1608X50N"
 			(at 116.84 34.29 0)
 			(effects
@@
 			)
 		)
-		(property "Footprint" "PCMTester2.0 Footprints:22uF_Capacitor"
+		(property "Footprint" "PCMFootprints:22uF_Capacitor"
 			(at 55.88 265.43 0)
 			(effects
@@
 			)
 		)
-		(property "Footprint" "PCMTester2.0 Footprints:22uF_Capacitor"
+		(property "Footprint" "PCMFootprints:22uF_Capacitor"
 			(at 48.26 111.76 0)
 			(effects
@@
 			)
 		)
-		(property "Footprint" "PCMTester2.0 Footprints:PWR_CORE1_footprint"
+		(property "Footprint" "PCMTester2.0_Footprints:PWR_CORE1_footprint"
 			(at 39.37 119.38 0)
 			(effects
@@
 			)
 		)
-		(property "Footprint" "PCMTester2.0 Footprints:SAMTEC_TSW-101-07-G-S (pin)"
+		(property "Footprint" "PCMFootprints:SAMTEC_TSW-101-07-G-S (pin)"
 			(at 356.87 114.3 0)
 			(effects
@@
 			)
 		)
-		(property "Footprint" "PCMTester2.0 Footprints:SAMTEC_TSW-101-07-G-S (pin)"
+		(property "Footprint" "PCMFootprints:SAMTEC_TSW-101-07-G-S (pin)"
 			(at 375.92 177.8 0)
 			(effects
@@
 			)
 		)
-		(property "Footprint" "PCMTester2.0 Footprints:22uF_Capacitor"
+		(property "Footprint" "PCMFootprints:22uF_Capacitor"
 			(at 35.56 83.82 0)
 			(effects
@@
 			)
 		)
-		(property "Footprint" "PCMTester2.0 Footprints:RESC1608X50N"
+		(property "Footprint" "PCMTester2.0_Footprints:RESC1608X50N"
 			(at 134.62 48.26 0)
 			(effects
@@
 			)
 		)
-		(property "Footprint" "PCMTester2.0 Footprints:SAMTEC_QTH-040-01-X-D-DP-A"
+		(property "Footprint" "PCMFootprints:SAMTEC_QTH-040-01-X-D-DP-A"
 			(at 455.93 104.14 0)
 			(effects
@@
 			)
 		)
-		(property "Footprint" "PCMTester2.0 Footprints:22uF_Capacitor"
+		(property "Footprint" "PCMFootprints:22uF_Capacitor"
 			(at 55.88 274.32 0)
 			(effects
@@
 			)
 		)
-		(property "Footprint" "PCMTester2.0 Footprints:SAMTEC_TSW-101-07-G-S (pin)"
+		(property "Footprint" "PCMFootprints:SAMTEC_TSW-101-07-G-S (pin)"
 			(at 267.97 177.8 0)
 			(effects
@@
 			)
 		)
-		(property "Footprint" "PCMTester2.0 Footprints:RESC1608X50N"
+		(property "Footprint" "PCMTester2.0_Footprints:RESC1608X50N"
 			(at 116.84 29.21 0)
 			(effects
@@
 			)
 		)
-		(property "Footprint" "PCMTester2.0 Footprints:TO_BM1_footprint"
+		(property "Footprint" "PCMTester2.0_Footprints:TO_BM1_footprint"
 			(at 110.49 232.41 0)
 			(effects
@@
 			)
 		)
-		(property "Footprint" "PCMTester2.0 Footprints:22uF_Capacitor"
+		(property "Footprint" "PCMFootprints:22uF_Capacitor"
 			(at 57.15 111.76 0)
 			(effects
@@
 			)
 		)
-		(property "Footprint" "PCMTester2.0 Footprints:RESC1608X50N"
+		(property "Footprint" "PCMTester2.0_Footprints:RESC1608X50N"
 			(at 134.62 63.5 0)
 			(effects
@@
 			)
 		)
-		(property "Footprint" "PCMTester2.0 Footprints:SAMTEC_QTH-040-01-X-D-DP-A"
+		(property "Footprint" "PCMFootprints:SAMTEC_QTH-040-01-X-D-DP-A"
 			(at 313.69 106.68 0)
 			(effects
@@
 			)
 		)
-		(property "Footprint" "PCMTester2.0 Footprints:RESC1608X50N"
+		(property "Footprint" "PCMTester2.0_Footprints:RESC1608X50N"
 			(at 134.62 53.34 0)
 			(effects
@@
 			)
 		)
-		(property "Footprint" "PCMTester2.0 Footprints:HRS_DF12NB-60DS-0.5V_51_"
+		(property "Footprint" "PCMFootprints:HRS_DF12NB-60DS-0.5V_51_"
 			(at 85.09 99.06 0)
 			(effects
@@
 			)
 		)
-		(property "Footprint" "PCMTester2.0 Footprints:RESC1608X50N"
+		(property "Footprint" "PCMTester2.0_Footprints:RESC1608X50N"
 			(at 134.62 58.42 0)
 			(effects
