File: PCMTester2.0/PCMTester2.0.kicad_pcb (KiCad board)
At the start: 2 copper layers, 150 x 150 mm, 21 parts

Commit message: added ground and power planes
Parts:
- turned C1 to 180 degrees
- turned C2 to 180 degrees
Routing:
- net GND: track 0.00 -> 54.9 mm, vias 0 -> 13
- net VDD: track 0.00 -> 23.3 mm, vias 0 -> 7
- net (no net): vias 0 -> 1
- added copper zone on In1.Cu, net GND
- added copper zone on In2.Cu, net VDD
Other:
- copper layers 2 -> 10
