File: PCMTester4.0/Map.kicad_sch (KiCad schematic)
At the start: 37 parts

Commit message: FINAL VERSION
Parts:
- removed NT11, NT14, NT15, NT21, NT22, NT31, NT32: ~, Library:Diff_Pair_Tie_swap_rev, symbol Library:Diff_Pair_Tie_swap
- removed NT13, NT19, NT20, NT26, NT27, NT28, NT29, NT30, NT5, NT7: ~, Library:Diff_Pair_Tie_swap, symbol Library:Diff_Pair_Tie_swap
- removed NT16, NT18, NT23, NT33, NT34, NT35, NT36, NT6: ~, Library:Diff_Pair_Tie_rev, symbol Library:Diff_Pair_Tie
- removed NT17, NT24, NT25, NT8: ~, Library:Diff_Pair_Tie, symbol Library:Diff_Pair_Tie

Commit message: ts buss
Other:
- note added: "unused | | V"
