File: PCMTester4.0/PCMTester4.0.kicad_sch (KiCad schematic)
At the start: 19 parts, among them J1 Phoenix MSTB 1x02 P5.08mm

Commit message: ts buss
Other:
- sheet CM connectors ports: added {DF12}, {FX11}; removed D{FC}, T{FC}, {DAQ_out}, {DAQ}, {TRIG_out}, {TRIG}
- sheet Map ports: added VDD, {DF12}, {FX11}; removed D{FC}, T{FC}, {DAQ_out}, {DAQ}, {TRIG_out}, {TRIG}
